File: hw/sch_pcb/USB232R02A/USB232R02A.kicad_sch (KiCad schematic)
At the start: 3 parts

Commit message: Edit
Parts:
- added C1: 10nF, Mlab_C:SMD-0805, symbol Device:C
- added C2: 10uF, Mlab_C:SMD-0805, symbol Device:C
- added C3, C4, C5: 100nF, Mlab_C:SMD-0805, symbol Device:C
- added D1: M4, Diode_SMD:D_SMA, symbol Device:D
- added D2: RED, Mlab_D:LED_1206, symbol Device:LED
- added D3: GREEN, Mlab_D:LED_1206, symbol Device:LED
- added FB1: BLM21PG300SN1D, Mlab_L:SMD-0805, symbol Device:FerriteBead_Small
- added H1, H2, H3, H4: M3, Mlab_Mechanical:dira_3mm, symbol Mechanical:MountingHole_Pad
- added J10, J11, J12, J13, J14, J15, J16, J4, J5, J6, J7, J8, J9: HEADER_2x01_PARALLEL, Mlab_Pin_Headers:Straight_2x01, symbol MLAB_HEADER:HEADER_2x01_PARALLEL
- added J2, J3: HEADER_2x03_PARALLEL, Mlab_Pin_Headers:Straight_2x03, symbol MLAB_HEADER:HEADER_2x03_PARALLEL
- added JP1: SolderJumper_2_Bridged, Jumper:SolderJumper-2_P1.3mm_Bridged_RoundedPad1.0x1.5mm, symbol Jumper:SolderJumper_2_Bridged
- added R1: 4k7, Mlab_R:SMD-0805, symbol Device:R
- added R2: 10k, Mlab_R:SMD-0805, symbol Device:R
- added R3, R4: 270R, Mlab_R:SMD-0805, symbol Device:R
- J1: renamed from J?; footprint (none) -> Connector_USB:USB_B_OST_USB-B1HSxx_Horizontal
- gave numbers to parts that had none: 2
Connections:
- net GND: now also U2.13 (GND), U2.21 (GND), U2.3 (GND), C1.2, C2.2, C3.2, C4.2, C5.1, D1.2 (A), H1.1, H2.1, H3.1, H4.1, J2.1, J2.2, J2.5, J2.6, J3.1, J3.2, J3.5, J3.6, R2.2
- net VBUS: now also C1.1, FB1.1
- net RXD: now reaches U2.1 (RXD)
- net RXD: now also J6.1, J6.2
- net +3V3: now reaches U2.10 (3V3OUT)
- net +3V3: now also C3.1, J3.3, J3.4, JP1.2 (B)
- net at U2.11 (~RESET): now also R1.2, R2.1
- net +5V: now reaches U2.12 (VCC)
- net +5V: now also C2.1, C4.1, D1.1 (K), D2.2 (A), D3.2 (A), FB1.2, J2.3, J2.4, R1.1
- net RXLED/CBUS1: now reaches U2.14 (CBUS1)
- net RXLED/CBUS1: now also J14.1, J14.2, R3.2
- net CBUS0: now reaches U2.15 (CBUS0)
- net CBUS0: now also J13.1, J13.2
- net CBUS3: now reaches U2.16 (CBUS3)
- net CBUS3: now also J16.1, J16.2
- net TXD: now reaches U2.17 (TXD)
- net TXD: now also J5.1, J5.2
- net #DTR: now reaches U2.18 (~DTR)
- net #DTR: now also J9.1, J9.2
- net #RTS: now reaches U2.19 (~RTS)
- net #RTS: now also J7.1, J7.2
- net #RI: now reaches U2.2 (~RI)
- net #RI: now also J12.1, J12.2
- net VCCIO: now reaches U2.20 (VCCIO)
- net VCCIO: now also C5.2, J4.1, J4.2, JP1.1 (A)
- net #DSR: now reaches U2.4 (~DSR)
- net #DSR: now also J10.1, J10.2
- net #DCD: now reaches U2.5 (~DCD)
- net #DCD: now also J11.1, J11.2
- net #CTS: now reaches U2.6 (~CTS)
- net #CTS: now also J8.1, J8.2
- net TXLED/CBUS2: now reaches U2.7 (CBUS2)
- net TXLED/CBUS2: now also J15.1, J15.2, R4.2
- new net: D3.1 (K), R4.1
- new net: D2.1 (K), R3.1
Other:
- note added: "CBUS Defaults CBUS0 - TXDEN CBUS1 - RXLED CBUS2 - TXLED CBUS3 - SLEEP#"
- moved on the sheet: J1, U1, U2
