File: hw/sch_pcb/USB232R02.kicad_sch (KiCad schematic)
At the start: 38 parts, among them J1 USB_B, J10 -, J11 -, J12 -, J13 -, J14 -, J15 -, J16 -, J17 HEADER_2x01_PARALLEL, J2 HEADER_2x03_PARALLEL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

Commit message: clean repo, update kicad footprints, prepare to assembly
Parts:
- removed J10, J11, J12, J4, J9: -, Mlab_Pin_Headers:Straight_2x01, symbol MLAB_HEADER:HEADER_2x01_PARALLEL
- removed J13, J14, J15, J16: -, Mlab_Pin_Headers:Straight_1x01, symbol MLAB_HEADER:HEADER_1x01
- removed J17, J5, J6, J7, J8: HEADER_2x01_PARALLEL, Mlab_Pin_Headers:Straight_2x01, symbol MLAB_HEADER:HEADER_2x01_PARALLEL
- added FID1, FID2: Fiducial, Fiducial:Fiducial_1mm_Mask2mm, symbol Mechanical:Fiducial
- added J18: HEADER_2x07, Mlab_Pin_Headers:Straight_2x07, symbol MLAB_HEADER:HEADER_2x07
- added J19: HEADER_2x05, Mlab_Pin_Headers:Straight_2x05, symbol MLAB_HEADER:HEADER_2x05_PARALLEL
- C1: LCSC (none) -> C913645
- C2: LCSC (none) -> C17024
- C3, C4, C5: LCSC (none) -> C111492
- D1: LCSC (none) -> C466506
- D2: footprint Mlab_D:LED_1206 -> Mlab_D:LED_1206_2; LCSC (none) -> C598398
- D3: footprint Mlab_D:LED_1206 -> Mlab_D:LED_1206_2; LCSC (none) -> C598394
- F1: LCSC (none) -> C269130
- FB1: LCSC (none) -> C16903
- H1, H2, H3, H4, JP1: now left out of the parts list
- J1: LCSC (none) -> C490687
- J2, J3: value HEADER_2x03_PARALLEL -> HEADER_2x03; LCSC (none) -> C706893
- R1: LCSC (none) -> C60816
- R2: LCSC (none) -> C84376
- R3, R4: LCSC (none) -> C228675
- U1: LCSC (none) -> C7519
- U2: LCSC (none) -> C132159
Connections:
- net #CTS: now also J19.5, J19.6
- net #DCD: now also J18.10, J18.9
- net #DSR: now also J18.7, J18.8
- net #DTR: now also J18.11, J18.12
- net #RI: now also J18.5, J18.6
- net #RTS: now also J19.7, J19.8
- net CBUS0: now also J18.4
- net CBUS3: now also J18.3
- net GND: now also J19.10, J19.9
- net RXD: now also J19.3, J19.4
- net RXLED/CBUS1: now also J18.2
- net TXD: now also J19.1, J19.2
- net TXLED/CBUS2: now also J18.1
- net VCCIO: now also J18.13, J18.14
- net DM renamed DN
Other:
- moved on the sheet: D2, D3, R3, R4

Commit message: aktualizace kodu a konfigurace
Parts:
- C1: LCSC C913645 -> C472806
Changed lines of the file:
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@@
       (effects (font (size 1.27 1.27)) hide)
     )
-    (property "LCSC" "C913645" (at 77.47 60.96 0)
+    (property "LCSC" "C472806" (at 77.47 60.96 0)
       (effects (font (size 1.27 1.27)) hide)
     )
